Commit message: finish grasping object

File: urdf/mobile_manipulator.urdf (robot description, URDF)
Before this commit: robot mobile_manipulator, 10 links, 9 joints
Links:
- added link vacuum_gripper, mass 0.0001; visual box size=0.05 0.1 0.021
Joints:
- added joint gripper_joint: type revolute, parent top_wrist, child vacuum_gripper, origin xyz=0.0 0 0.13 rpy=0 0 0, axis 0 1 0, limit lower=0 upper=0 effort=50 velocity=10
- joint top_wrist_joint: type continous -> continuous
